File: InputModule.kicad_sch (KiCad schematic)
At the start: 20 parts, among them J7 Volume Control, J8 Muting Control, K1 EC2-5NU, U5 TL072

Commit message: Update footprints
Parts:
- C15, C16: footprint (none) -> Capacitor_THT:C_Radial_D6.3mm_H11.0mm_P2.50mm
- C17, C18: footprint (none) -> Capacitor_THT:C_Rect_L7.0mm_W2.5mm_P5.00mm
- C19, C20: footprint (none) -> Capacitor_THT:C_Rect_L10.3mm_W4.5mm_P7.50mm_MKS4
- U5: footprint (none) -> Package_DIP:DIP-8_W7.62mm_Socket
Changed lines of the file:
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@@
     (property "Reference" "U5" (id 0) (at 124.46 76.2 0))
     (property "Value" "TL072" (id 1) (at 124.46 73.66 0))
-    (property "Footprint" "" (id 2) (at 124.46 66.04 0)
+    (property "Footprint" "Package_DIP:DIP-8_W7.62mm_Socket" (id 2) (at 124.46 66.04 0)
       (effects (font (size 1.27 1.27)) hide)
     )
@@
     (property "Reference" "C20" (id 0) (at 201.93 73.66 90))
     (property "Value" "0.2u" (id 1) (at 201.93 76.2 90))
-    (property "Footprint" "" (id 2) (at 205.74 80.3148 0)
+    (property "Footprint" "Capacitor_THT:C_Rect_L10.3mm_W4.5mm_P7.50mm_MKS4" (id 2) (at 205.74 80.3148 0)
       (effects (font (size 1.27 1.27)) hide)
     )
@@
     (property "Reference" "C15" (id 0) (at 100.33 54.61 90))
     (property "Value" "22u" (id 1) (at 100.33 57.15 90))
-    (property "Footprint" "" (id 2) (at 104.14 61.2648 0)
+    (property "Footprint" "Capacitor_THT:C_Radial_D6.3mm_H11.0mm_P2.50mm" (id 2) (at 104.14 61.2648 0)
       (effects (font (size 1.27 1.27)) hide)
     )
@@
     (property "Reference" "C17" (id 0) (at 124.46 35.56 90))
     (property "Value" "47p" (id 1) (at 124.46 38.1 90))
-    (property "Footprint" "" (id 2) (at 128.27 42.2148 0)
+    (property "Footprint" "Capacitor_THT:C_Rect_L7.0mm_W2.5mm_P5.00mm" (id 2) (at 128.27 42.2148 0)
       (effects (font (size 1.27 1.27)) hide)
     )
@@
     (property "Reference" "U5" (id 0) (at 124.46 118.11 0))
     (property "Value" "TL072" (id 1) (at 124.46 115.57 0))
-    (property "Footprint" "" (id 2) (at 124.46 107.95 0)
+    (property "Footprint" "Package_DIP:DIP-8_W7.62mm_Socket" (id 2) (at 124.46 107.95 0)
       (effects (font (size 1.27 1.27)) hide)
     )
@@
     (property "Reference" "C19" (id 0) (at 201.93 58.42 90))
     (property "Value" "0.2u" (id 1) (at 201.93 60.96 90))
-    (property "Footprint" "" (id 2) (at 205.74 65.0748 0)
+    (property "Footprint" "Capacitor_THT:C_Rect_L10.3mm_W4.5mm_P7.50mm_MKS4" (id 2) (at 205.74 65.0748 0)
       (effects (font (size 1.27 1.27)) hide)
     )
@@
     (property "Reference" "C18" (id 0) (at 124.46 78.74 90))
     (property "Value" "47p" (id 1) (at 124.46 81.28 90))
-    (property "Footprint" "" (id 2) (at 128.27 85.3948 0)
+    (property "Footprint" "Capacitor_THT:C_Rect_L7.0mm_W2.5mm_P5.00mm" (id 2) (at 128.27 85.3948 0)
       (effects (font (size 1.27 1.27)) hide)
     )
@@
     (property "Reference" "C16" (id 0) (at 101.6 96.52 90))
     (property "Value" "22u" (id 1) (at 101.6 99.06 90))
-    (property "Footprint" "" (id 2) (at 105.41 103.1748 0)
-      (effects (font (size 1.27 1.27)) hide)
-    )
+    (property "Footprint" "Capacitor_THT:C_Radial_D6.3mm_H11.0mm_P2.50mm" (id 2) (at 105.41 103.1748 0)
+      (effects (font (size 1.27 1.27)) hide)
+    )

Commit message: Finalize schematic and start with PCB layout
Parts:
- removed C19, C20: 0.2u, Capacitor_THT:C_Rect_L10.3mm_W4.5mm_P7.50mm_MKS4, symbol Device:C
- removed R10, R9: 22K, symbol Device:R
- added C31, C32: 10u, Capacitor_THT:C_Rect_L10.3mm_W4.5mm_P7.50mm_MKS4, symbol Device:C
- added D3: DIODE, Diode_THT:D_DO-34_SOD68_P7.62mm_Horizontal, symbol pspice:DIODE
- added R21, R22: 22K, Resistor_THT:R_Axial_DIN0207_L6.3mm_D2.5mm_P10.16mm_Horizontal, symbol Device:R
- C27: renamed from C15; value 22u -> 10u
- C28: renamed from C16; value 22u -> 10u
- J11: renamed from J7; footprint (none) -> Connector_PinHeader_2.54mm:PinHeader_1x05_P2.54mm_Vertical
- J12: renamed from J8; footprint (none) -> Connector_JST:JST_EH_B2B-EH-A_1x02_P2.50mm_Vertical
- K3: renamed from K1; footprint Relay_THT:Relay_DPDT_Kemet_EC2 -> Relay_THT:Relay_DPDT_Omron_G5V-2; symbol Relay:EC2-5NU -> Relay:G5V-2
- R17: renamed from R5; footprint (none) -> Resistor_THT:R_Axial_DIN0207_L6.3mm_D2.5mm_P10.16mm_Horizontal
- R18: renamed from R6; footprint (none) -> Resistor_THT:R_Axial_DIN0207_L6.3mm_D2.5mm_P10.16mm_Horizontal
- R19: renamed from R7; footprint (none) -> Resistor_THT:R_Axial_DIN0207_L6.3mm_D2.5mm_P10.16mm_Horizontal
- R20: renamed from R8; footprint (none) -> Resistor_THT:R_Axial_DIN0207_L6.3mm_D2.5mm_P10.16mm_Horizontal
- RV5: renamed from RV1; footprint (none) -> Potentiometer_THT:Potentiometer_Bourns_3266Z_Horizontal
- RV6: renamed from RV2; footprint (none) -> Potentiometer_THT:Potentiometer_Bourns_3266Z_Horizontal
- renumbered #RV1 to #RV5, #RV2 to #RV6, C17 to C29, C18 to C30, U5 to U4
Connections:
- net GND: now also #RV6.3, K3.11, K3.6; no longer #RV6.1, K3.10, K3.3
- net GND2: now also K3.16, D3.1 (K); no longer K3.12
- net L Out: now also R21.2; no longer K3.5
- net R Out: now also R22.2; no longer K3.8
- net at #RV5.1, J11.5 (Pin_5): now also C32.2
- net at #RV5.2, J11.4 (Pin_4): now also K3.13
- net at C30.2, RV6.2, U4.7: now also C32.1
- net at J12.2 (Pin_2), K3.1: now also D3.2 (A)
- net at #RV6.2, J11.2 (Pin_2): now also K3.4
- net at J11.1 (Pin_1): now also #RV6.1, C31.2; no longer #RV6.3
- net at C29.2, RV5.2, U4.1: now also C31.1
- net at K3.9: now also R22.1
- new net: K3.8, R21.1
Other:
- moved on the sheet: J12
